File: esp32-S3 fully intergrated main board/motorcontrol.kicad_sch (KiCad schematic)
At the start: 25 parts, among them J2 Conn_01x03_Pin, Q1 BUK7M6R3-40EX, Q2 BUK7M6R3-40EX, Q4 BUK7M6R3-40EX, Q5 BUK7M6R3-40EX, Q8 BUK7M6R3-40EX, Q9 BUK7M6R3-40EX, U2 IR2133S

Commit message: fixing ic
Parts:
- removed C13, C2, C3, C4: 100u, symbol Device:C_Polarized
- removed C5: C, symbol Device:C
- removed D1, D2, D3: D, symbol Device:D
- removed R2, R3, R4, R5, R6, R9: 47R, symbol Device:R
- removed U2: IR2133S, Package_SO:SOIC-28W_7.5x17.9mm_P1.27mm, symbol Driver_FET:IR2133S
- added R1: R, symbol Device:R
- added U5: ~, symbol project:6EDL7151
Connections:
- net GND: now also R1.2, U5.17 (PGND), U5.49 (GND); no longer Q9.1 (S), Q9.2 (S), Q9.3 (S)
- net at Q8.4 (G): now also U5.25 (GHC)
- new net: Q9.1 (S), Q9.2 (S), Q9.3 (S), R1.1, U5.29 (SLC)
Other:
- moved on the sheet: J2, Q1, Q2, Q4, Q5, Q8, Q9, R21, R8
